File: KICAD8/COMMIT_5/H.A.V.O.C. PCB V 1.0.kicad_pcb (KiCad board)
At the start: 8 copper layers, 65 x 100 mm, 129 parts, among them IC2 STM32H755IIT6, J10 Conn_02x10_Top_Bottom, J2 USB_B_Micro, J3 XT60-M, J5 Conn_Coaxial, J6 Conn_Coaxial, J7 Conn_02x10_Top_Bottom, M1 SERVO1, M2 SERVO2, M3 SERVO3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

Commit message: Removed signal traces from 3v3 power plane. Connected (hopefully) all gnd connections. Rerouted other miscilaneous traces.
Routing:
- net GND: track 159.9 -> 222.0 mm, vias 113 -> 120
- net SERVO1: track 45.8 -> 87.7 mm
- net USB_D+: track 50.9 -> 81.4 mm
- net USB_D-: track 50.8 -> 75.7 mm, vias 3 -> 2
- net +3V3: track 125.0 -> 144.7 mm
- net GP_GPIO34: track 101.8 -> 91.2 mm
- net Net-(5VReg1-EN): track 43.4 -> 48.6 mm, vias 2 -> 1
- net SPI1_SCK: track 11.3 -> 14.1 mm
- net +5V: track 188.5 -> 185.7 mm
- net Net-(3v3Reg1-SW): track 14.7 -> 17.0 mm
- net V_DETECT: track 10.6 -> 12.7 mm, vias 2 -> 0
- net GP_GPIO20: track 42.3 -> 43.7 mm
- net UART5_TX: track 58.8 -> 57.9 mm
- net SPI2_MISO: track 18.8 -> 19.6 mm
- net GP_GPIO10: track 45.2 -> 45.9 mm
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